File: integrator.sch (KiCad schematic (older format))
At the start: 21 parts, among them J1 SJ-3524-SMT, J2 SJ-3524-SMT, SW1 EVQP40B3M, SW2 EVQP40B3M, SW3 SW_Push_LED, U1 Teensy3.2, U2 ICM-42605

Commit message: version 5 schematic complete
Parts:
- removed C1: 10nf, Capacitor_SMD:C_0805_2012Metric, symbol Device:C_Small
- removed C2: 0.1uf, Capacitor_SMD:C_0805_2012Metric, symbol Device:C_Small
- removed C3: 2.2uf, Capacitor_SMD:C_0805_2012Metric, symbol Device:C_Small
- removed C4, C6: 4.7uf, Capacitor_SMD:CP_Elec_5x4.5, symbol Device:C_Small
- removed D1: SD0805S020S1R0, Diode_SMD:D_0805_2012Metric, symbol Device:D_Schottky_Small
- removed R1, R2: 47, Resistor_SMD:R_0805_2012Metric, symbol Device:R
- removed SW3: SW_Push_LED, TL3215AF160BQ:E-Switch-N326000-0-0-0, symbol TL3215AF160BQ:TL3215AF160BQ
- removed U1: Teensy3.2, teensy:Teensy30_31_32_LC, symbol teensy:Teensy3.2
- removed U2: ICM-42605, ICM-42605:PQFN50P300X250X97-14N, symbol ICM-42605:ICM-42605
- added C? (x2): 9pf, Capacitor_SMD:C_0805_2012Metric, symbol Device:C_Small
- added C? (x8): 0.1uf, Capacitor_SMD:C_0805_2012Metric, symbol Device:C_Small
- added C?: 1nf, Capacitor_SMD:C_0805_2012Metric, symbol Device:C_Small
- added C?: 10nf, Capacitor_SMD:C_0805_2012Metric, symbol Device:C_Small
- added C?: 2.2uf, Capacitor_SMD:C_0805_2012Metric, symbol Device:C_Small
- added C?: 4.7uf, Capacitor_SMD:C_0805_2012Metric, symbol Device:C_Small
- added D?: <300mv drop, symbol Device:D_Schottky_Small
- added D?: 900mv drop, symbol Device:D_Schottky_Small
- added J?: Conn_ARM_JTAG_SWD_10, symbol Connector:Conn_ARM_JTAG_SWD_10
- added J?: USB_C_Receptacle_USB2.0, symbol Connector:USB_C_Receptacle_USB2.0
- added J? (x2): SP-3533-02, CUI_SP-3533-02, symbol SP-3533-02:SP-3533-02
- added L?: 10uh, symbol Device:L
- added LED? (x2): LS_L29K-G1J2-1-Z, LED_SMD:LED_0805_2012Metric, symbol 2021-01-16_04-43-04:LS_L29K-G1J2-1-Z
- added R?: 5,1k, Resistor_SMD:R_0805_2012Metric, symbol Device:R
- added R?: 5.1k, Resistor_SMD:R_0805_2012Metric, symbol Device:R
- added R?: 1, Resistor_SMD:R_0805_2012Metric, symbol Device:R
- added R? (x2): 10k, Resistor_SMD:R_0805_2012Metric, symbol Device:R
- added R? (x2): 27 5%, Resistor_SMD:R_0805_2012Metric, symbol Device:R
- added SW?: EVQP40B3M, Button_Switch_THT:ksa0v311 lftr, symbol edgesw:EVQP40B3M
- added SW?: 436333033816, symbol Switch:436333033816
- added U?: ATSAM4S8BB-MN, MODULE, symbol ATSAM4S8BB-MN:ATSAM4S8BB-MN
- added U?: LSM6DSO32XTR, LGA_O32XTR_STM, symbol 2022-04-26_22-02-23:LSM6DSO32XTR
- added U?: MCP1501T-18E_RW, WDFN8_RW_MCH, symbol 2022-05-07_05-34-42:MCP1501T-18E_RW
- added U?: TC1263-3.3VOATR, Microchip-TC1263-3.3VOATR-*, symbol tc1263:TC1263-3.3VOATR
- added Y?: Crystal, symbol Device:Crystal
- R4, R5: value 5k -> 10k
Connections:
- net labels added: AGnd, VReg, po_swclk, po_swdio, po_swo, ring1_io, ring2_io, tip1_io, tip2_in, tip2_io, tip2_out
- net labels removed: +3.3v, a_gnd, dac, l_sync_out, r_sync_out, spi_cs, sw1, sw2, swclk, swdio, swo
- wire segments 154 -> 252
Other:
- moved on the sheet: J1, J2, R4, R5, R6

Commit message: rev5 pcb checkpoint (close)
Parts:
- removed J?: USB_C_Receptacle_USB2.0, symbol Connector:USB_C_Receptacle_USB2.0
- added C15: 100uf, Capacitor_SMD:CP_Elec_6.3x5.2, symbol Device:C_Small
- added C16: 100uf(NC), Capacitor_SMD:CP_Elec_6.3x5.2, symbol Device:C_Small
- added J5: USB4105-GF-A, GCT_USB4105-GF-A, symbol usb4105:USB4105-GF-A
- D1: renamed from D?; footprint (none) -> Diode_SMD:D_TUMD2
- D2: renamed from D?; footprint (none) -> Diode_SMD:D_0201_0603Metric
- J3, J4: renamed from J?; footprint CUI_SP-3533-02 -> SP-3533-02:CUI_SP-3533-02
- J6: renamed from J?; footprint (none) -> Connector_PinHeader_2.54mm:PinHeader_2x05_P2.54mm_Horizontal
- L1: renamed from L?; footprint (none) -> Inductor_SMD:L_0805_2012Metric
- SW1, SW2: footprint Button_Switch_THT:ksa0v311 lftr -> tl1105:TL1105VF100Q
- SW3: renamed from SW?; footprint Button_Switch_THT:ksa0v311 lftr -> tl1105:TL1105VF100Q
- SW4: renamed from SW?; footprint (none) -> misc:436333033816
- U1: renamed from U?; footprint WDFN8_RW_MCH -> MCP1501T-18E-RW:MCP1501T-18E&slash_RW
- U2: renamed from U?; footprint Microchip-TC1263-3.3VOATR-* -> tc1263:Microchip-TC1263-3.3VOATR-Level_A
- U3: renamed from U?; footprint LGA_O32XTR_STM -> LSM6DSO32XTR:LSM6DSO32XTR
- U4: renamed from U?; footprint MODULE -> Package_DFN_QFN:QFN-64-1EP_9x9mm_P0.5mm_EP6x6mm_ThermalVias
- Y1: renamed from Y?; footprint (none) -> tsx-3225:TSX-3225; symbol Device:Crystal -> tsx-3225:TSX-3225
- gave numbers to parts that had none: 23
Connections:
- net labels added: advref, led3, led4, ring1, ring2, spi_cs, tip1, tip2, usb_dneg, usb_dpos, usb_vbus, vddin, vddout
- net labels removed: tip2_in, tip2_out
- wire segments 252 -> 304
Other:
- moved on the sheet: C13, C14, R6

Commit message: v5 sent to fab
Parts:
- added C17: 1uf, Capacitor_SMD:C_0805_2012Metric, symbol Device:C_Small
- added J7: test point, Connector_PinHeader_2.54mm:PinHeader_2x02_P2.54mm_Vertical, symbol Connector_Generic:Conn_02x02_Counter_Clockwise
- J5: footprint GCT_USB4105-GF-A -> usb4105:GCT_USB4105-GF-A
- POGO1: symbol Connector_Generic_MountingPin:Conn_02x06_Odd_Even_MountingPin -> Connector_Generic:Conn_02x06_Odd_Even
Connections:
- wire segments 304 -> 322
Other:
- moved on the sheet: D1, D2
Changed lines of the file:
@@
 $EndComp
 $Comp
-L Connector_Generic_MountingPin:Conn_02x06_Odd_Even_MountingPin POGO1
+L Connector_Generic:Conn_02x06_Odd_Even POGO1
 U 1 1 6011B68E
 P 14600 5800
@@
 $EndComp
 $Comp
-L Device:D_Schottky_Small D1
-U 1 1 6278B65C
-P 14300 7150
-F 0 "D1" H 14350 7350 50  0000 R CNN
-F 1 "<300mv drop" H 14550 7250 50  0000 R CNN
-F 2 "Diode_SMD:D_TUMD2" V 14300 7150 50  0001 C CNN
-F 3 "~" V 14300 7150 50  0001 C CNN
-	1    14300 7150
-	0    -1   -1   0
-$EndComp
-$Comp
 L Device:D_Schottky_Small D2
 U 1 1 6278CCAC
-P 14550 7150
-F 0 "D2" H 14550 7350 50  0000 C CNN
-F 1 "900mv drop" H 14550 7250 50  0000 C CNN
-F 2 "Diode_SMD:D_0201_0603Metric" V 14550 7150 50  0001 C CNN
-F 3 "~" V 14550 7150 50  0001 C CNN
-	1    14550 7150
+P 14700 7350
+F 0 "D2" H 14700 7550 50  0000 C CNN
+F 1 "900mv drop" H 14700 7450 50  0000 C CNN
+F 2 "Diode_SMD:D_0201_0603Metric" V 14700 7350 50  0001 C CNN
+F 3 "~" V 14700 7350 50  0001 C CNN
+	1    14700 7350
 	0    1    1    0
 $EndComp
@@
 VReg
 Wire Wire Line
-	14550 7050 14550 6650
-Wire Wire Line
-	14550 6650 14400 6650
-Wire Wire Line
-	14550 7250 14550 7600
-Wire Wire Line
-	14550 7600 14400 7600
+	14700 7250 14700 7200
+Wire Wire Line
+	14700 7450 14700 7600
 Wire Wire Line
 	14400 7600 14400 7700
 Wire Wire Line
-	14300 7250 14300 7600
-Wire Wire Line
-	14300 7600 14400 7600
-Connection ~ 14400 7600
-Wire Wire Line
-	14300 7050 14300 6650
-Wire Wire Line
 	14400 6100 14400 6650
-Connection ~ 14400 6650
-Wire Wire Line
-	14300 6650 14400 6650
 $Comp
 L power:Earth #PWR0109
@@
 	6000 6700 6700 6700
 Connection ~ 6000 6550
-Wire Wire Line
-	10800 7400 13750 7400
 Wire Wire Line
 	14900 5800 15600 5800
@@
 	-1   0    0    1
 $EndComp
-Wire Wire Line
-	4000 6350 4000 6000
 Connection ~ 4000 6350
 Wire Wire Line
@@
 Wire Wire Line
 	3700 5800 4000 5800
-Wire Wire Line
-	3700 5800 2950 5800
-Connection ~ 3700 5800
 Text Label 13750 1800 1    50   ~ 0
 tip2
@@
 F 0 "J5" H 1450 8367 50  0000 C CNN
 F 1 "USB4105-GF-A" H 1450 8276 50  0000 C CNN
-F 2 "GCT_USB4105-GF-A" H 1450 7700 50  0001 L BNN
+F 2 "usb4105:GCT_USB4105-GF-A" H 1450 7700 50  0001 L BNN
 F 3 "" H 1450 7700 50  0001 L BNN
 F 4 "A3" H 1450 7700 50  0001 L BNN "PARTREV"
@@
 Wire Wire Line
 	8100 8750 8100 8400
+Wire Wire Line
+	14100 6650 14400 6650
+Wire Wire Line
+	14100 6750 14100 6650
+Wire Wire Line
+	14100 7600 14400 7600
+Wire Wire Line
+	14100 6950 14100 7100
+$Comp
+L Device:D_Schottky_Small D1
+U 1 1 6278B65C
+P 14100 6850
+F 0 "D1" H 14150 7050 50  0000 R CNN
+F 1 "<300mv drop" H 14350 6950 50  0000 R CNN
+F 2 "Diode_SMD:D_TUMD2" V 14100 6850 50  0001 C CNN
+F 3 "~" V 14100 6850 50  0001 C CNN
+	1    14100 6850
+	0    -1   -1   0
+$EndComp
+Wire Wire Line
+	10800 7400 13750 7400
+$Comp
+L Connector_Generic:Conn_02x02_Counter_Clockwise J7
+U 1 1 62BDDB43
+P 14450 7200
+F 0 "J7" H 14500 6875 50  0000 C CNN
+F 1 "test point" H 14500 6966 50  0000 C CNN
+F 2 "Connector_PinHeader_2.54mm:PinHeader_2x02_P2.54mm_Vertical" H 14450 7200 50  0001 C CNN
+F 3 "~" H 14450 7200 50  0001 C CNN
+	1    14450 7200
+	-1   0    0    1
+$EndComp
+Wire Wire Line
+	14400 6650 14700 6650
+Connection ~ 14400 6650
+Wire Wire Line
+	14400 7600 14700 7600
+Connection ~ 14400 7600
+Wire Wire Line
+	14150 7100 14100 7100
+Connection ~ 14100 7100
+Wire Wire Line
+	14100 7100 14100 7200
+Wire Wire Line
+	14150 7200 14100 7200
+Connection ~ 14100 7200
+Wire Wire Line
+	14100 7200 14100 7600
+Wire Wire Line
+	14650 7100 14700 7100
+Connection ~ 14700 7100
+Wire Wire Line
+	14700 7100 14700 6650
+Wire Wire Line
+	14650 7200 14700 7200
+Connection ~ 14700 7200
+Wire Wire Line
+	14700 7200 14700 7100
+Wire Wire Line
+	900  800  900  700
+Wire Wire Line
+	900  700  1500 700
+Wire Wire Line
+	1500 700  1500 800
+Wire Wire Line
+	1000 800  1000 650
+Wire Wire Line
+	1000 650  1600 650
+Wire Wire Line
+	1600 650  1600 800
+Wire Wire Line
+	1100 800  1100 600
+Wire Wire Line
+	1100 600  1700 600
+Wire Wire Line
+	1700 600  1700 800
+$Comp
+L Device:C_Small C17
+U 1 1 627DC005
+P 4100 6050
+F 0 "C17" H 4192 6096 50  0000 L CNN
+F 1 "1uf" H 4192 6005 50  0000 L CNN
+F 2 "Capacitor_SMD:C_0805_2012Metric" H 4100 6050 50  0001 C CNN
+F 3 "~" H 4100 6050 50  0001 C CNN
+	1    4100 6050
+	0    1    1    0
+$EndComp
+$Comp
+L power:Earth #PWR01
+U 1 1 627DD4E3
+P 4300 5950
+F 0 "#PWR01" H 4300 5700 50  0001 C CNN
+F 1 "Earth" H 4300 5800 50  0001 C CNN
+F 2 "" H 4300 5950 50  0000 C CNN
+F 3 "" H 4300 5950 50  0000 C CNN
+	1    4300 5950
+	-1   0    0    1
+$EndComp
+Wire Wire Line
+	4200 6050 4300 5950
+Connection ~ 4000 6050
+Wire Wire Line
+	4000 6050 4000 6000
+Wire Wire Line
+	4000 6050 4000 6350
 $EndSCHEMATC

Commit message: tweaks/fixes to v5
Parts:
- added SW5: 436333033816, misc:436333033816, symbol Switch:436333033816
- D2: footprint Diode_SMD:D_0201_0603Metric -> Diode_SMD:D_0603_1608Metric
Connections:
- wire segments 322 -> 331
Changed lines of the file:
@@
 	1    0    0    -1
 $EndComp
-Text Label 14900 6400 3    50   ~ 0
+Text Label 14950 6100 3    50   ~ 0
 po_play
 Text Label 14400 6250 3    50   ~ 0
@@
 F 0 "D2" H 14700 7550 50  0000 C CNN
 F 1 "900mv drop" H 14700 7450 50  0000 C CNN
-F 2 "Diode_SMD:D_0201_0603Metric" V 14700 7350 50  0001 C CNN
+F 2 "Diode_SMD:D_0603_1608Metric" V 14700 7350 50  0001 C CNN
 F 3 "~" V 14700 7350 50  0001 C CNN
 	1    14700 7350
@@
 Wire Wire Line
 	4000 6050 4000 6350
+$Comp
+L Switch:436333033816 SW5
+U 1 1 62BD359C
+P 4650 8400
+F 0 "SW5" V 4650 7992 50  0000 R CNN
+F 1 "436333033816" H 4650 8900 50  0001 C CNN
+F 2 "misc:436333033816" H 4600 7950 50  0001 C CNN
+F 3 "" H 4600 7950 50  0001 C CNN
+	1    4650 8400
+	1    0    0    -1
+$EndComp
+Connection ~ 5000 8750
+Wire Wire Line
+	4300 8750 4300 8200
+Wire Wire Line
+	4300 8200 4400 8200
+Connection ~ 4300 8750
+Wire Wire Line
+	4900 8200 5000 8200
+Wire Wire Line
+	5000 8200 5000 8750
+Wire Wire Line
+	8900 5300 8900 3550
+Wire Wire Line
+	8900 3550 4650 3550
+Wire Wire Line
+	4650 3550 4650 8200
+Wire Wire Line
+	4300 8750 5000 8750
+Text GLabel 4100 8750 0    50   Input ~ 0
+VReg
+Wire Wire Line
+	4100 8750 4300 8750
 $EndSCHEMATC

Commit message: major cleanup/reorg of symbols and footprints
Parts:
- LED1, LED2, LED3, LED4: symbol 2021-01-16_04-43-04:LS_L29K-G1J2-1-Z -> integrator-rescue:LS_L29K-G1J2-1-Z-2021-01-16_04-43-04
- SW1, SW2, SW3: symbol edgesw:EVQP40B3M -> integrator-rescue:EVQP40B3M-edgesw
- U1: symbol 2022-05-07_05-34-42:MCP1501T-18E_RW -> integrator-rescue:MCP1501T-18E_RW-2022-05-07_05-34-42
- U3: symbol 2022-04-26_22-02-23:LSM6DSO32XTR -> integrator-rescue:LSM6DSO32XTR-2022-04-26_22-02-23
Changed lines of the file:
@@
 $EndComp
 $Comp
-L edgesw:EVQP40B3M SW1
+L integrator-rescue:EVQP40B3M-edgesw SW1
 U 1 1 5FECB177
 P 3000 3850
@@
 $EndComp
 $Comp
-L edgesw:EVQP40B3M SW2
+L integrator-rescue:EVQP40B3M-edgesw SW2
 U 1 1 5FECB345
 P 14100 2750
@@
 spi_mosi
 $Comp
-L edgesw:EVQP40B3M SW3
+L integrator-rescue:EVQP40B3M-edgesw SW3
 U 1 1 62687826
 P 8100 1550
@@
 $EndComp
 $Comp
-L 2021-01-16_04-43-04:LS_L29K-G1J2-1-Z LED2
+L integrator-rescue:LS_L29K-G1J2-1-Z-2021-01-16_04-43-04 LED2
 U 1 1 6002719A
 P 14400 1050
@@
 $EndComp
 $Comp
-L 2021-01-16_04-43-04:LS_L29K-G1J2-1-Z LED3
+L integrator-rescue:LS_L29K-G1J2-1-Z-2021-01-16_04-43-04 LED3
 U 1 1 626E52CF
 P 8150 950
@@
 $EndComp
 $Comp
-L 2022-04-26_22-02-23:LSM6DSO32XTR U3
+L integrator-rescue:LSM6DSO32XTR-2022-04-26_22-02-23 U3
 U 1 1 6275887D
 P 3450 9700
@@
 	11550 8500 11550 8850
 $Comp
-L 2021-01-16_04-43-04:LS_L29K-G1J2-1-Z LED4
+L integrator-rescue:LS_L29K-G1J2-1-Z-2021-01-16_04-43-04 LED4
 U 1 1 62795B7F
 P 11550 8100
@@
 	1100 4900 1300 4900
 $Comp
-L 2022-05-07_05-34-42:MCP1501T-18E_RW U1
+L integrator-rescue:MCP1501T-18E_RW-2022-05-07_05-34-42 U1
 U 1 1 62781FDF
 P 1300 4900
@@
 $EndComp
 $Comp
-L 2021-01-16_04-43-04:LS_L29K-G1J2-1-Z LED1
+L integrator-rescue:LS_L29K-G1J2-1-Z-2021-01-16_04-43-04 LED1
 U 1 1 60027292
 P 3700 2100

Commit message: WIP
Parts:
- removed C5, C7, C8: 0.1uf, Capacitor_SMD:C_0805_2012Metric, symbol Device:C_Small
- removed C6: 2.2uf, Capacitor_SMD:C_0805_2012Metric, symbol Device:C_Small
- removed U2: TC1263-3.3VOATR, tc1263:Microchip-TC1263-3.3VOATR-Level_A, symbol tc1263:TC1263-3.3VOATR
- removed U4: ATSAM4S8BB-MN, Package_DFN_QFN:QFN-64-1EP_9x9mm_P0.5mm_EP6x6mm_ThermalVias, symbol ATSAM4S8BB-MN:ATSAM4S8BB-MN
- added C? (x2): 10uf, Capacitor_SMD:C_0805_2012Metric, symbol Device:C_Small
- added D?: 900mv drop, Diode_SMD:D_0603_1608Metric, symbol Device:D_Schottky_Small
- added R?: 1k 5%, Resistor_SMD:R_0805_2012Metric, symbol Device:R
- added U?: RP2040, IC57_RP2040, symbol RP2040:RP2040
- added U?: ISL9110, symbol Power_Management:ISL9110
- L1: value 10uh -> 2.2uh
- U1: footprint MCP1501T-18E-RW:MCP1501T-18E&slash_RW -> WDFN8_RW_MCH; symbol integrator-rescue:MCP1501T-18E_RW-2022-05-07_05-34-42 -> MCP1501T:MCP1501T-18E_RW
- U3: symbol integrator-rescue:LSM6DSO32XTR-2022-04-26_22-02-23 -> LSM6DSO32XTR:LSM6DSO32XTR
- Y1: footprint tsx-3225:TSX-3225 -> misc:XTAL_ABLS-12.000MHZ-B4-T; symbol tsx-3225:TSX-3225 -> ABLS-12.000MHZ-B4-T:ABLS-12.000MHZ-B4-T
Connections:
- net labels added: VRaw
- net labels removed: vddin, vddout
- wire segments 331 -> 277
Other:
- moved on the sheet: C1, C10, C11, C12, C15, C16, C17, C3, C9, J1, L1, LED1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

Commit message: WIP
Parts:
- removed C10, C14: 0.1uf, Capacitor_SMD:C_0805_2012Metric, symbol Device:C_Small
- removed C13: 10nf, Capacitor_SMD:C_0805_2012Metric, symbol Device:C_Small
- removed C15: 100uf, Capacitor_SMD:CP_Elec_6.3x5.2, symbol Device:C_Small
- removed C16: 100uf(NC), Capacitor_SMD:CP_Elec_6.3x5.2, symbol Device:C_Small
- removed C17: 1uf, Capacitor_SMD:C_0805_2012Metric, symbol Device:C_Small
- removed C9: 4.7uf, Capacitor_SMD:C_0805_2012Metric, symbol Device:C_Small
- removed R9: 1, Resistor_SMD:R_0805_2012Metric, symbol Device:R
- removed SW5: 436333033816, misc:436333033816, symbol Switch:436333033816
- added C? (x2): 1uf, Capacitor_SMD:C_0805_2012Metric, symbol Device:C_Small
- added C? (x11): 0.1uf, Capacitor_SMD:C_0805_2012Metric, symbol Device:C_Small
- added R?: 10k, Resistor_SMD:R_0805_2012Metric, symbol Device:R
- added R?: 1k, Resistor_SMD:R_0805_2012Metric, symbol Device:R
- added U?: W25Q128JVS, Package_SO:SOIC-8_5.23x5.23mm_P1.27mm, symbol Memory_Flash:W25Q128JVS
- C11, C12: value 9pf -> 27pf
- J5: Note (none) -> USB-C Connector
Connections:
- net labels added: VAref, VInt, imu_int, pi_reset, pi_swclk, pi_swdio, sw1, sw2, sw3, sw4, usb_boot
- net labels removed: advref, imu_int1, nonstop_led, nonstop_sw, ring1_io, ring2_io, tip1_io, tip2_io, usb_vbus
- wire segments 277 -> 286
Other:
- moved on the sheet: C1, C11, C12, C3, C?, D?, J1, J2, J3, J4, J5, J6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

Commit message: WIP before schematic append
Parts:
- added C14, C15: 47u, Capacitor_SMD:C_0805_2012Metric, symbol Device:C
- added C4, C7, C8: 100n, Capacitor_SMD:C_0402_1005Metric, symbol Device:C
- added R1, R2: 220, Resistor_SMD:R_0402_1005Metric, symbol Device:R
- added R3, R4: 100, Resistor_SMD:R_0402_1005Metric, symbol Device:R
- added R7, R8: 1.8K, Resistor_SMD:R_0402_1005Metric, symbol Device:R
- U1: value MCP1501T-18E_RW -> MCP1501T-30E_RW
Connections:
- net labels added: +3.3VA, GND, PWM_AUDIO_L, PWM_AUDIO_R, PWM_L, PWM_LL, PWM_R, PWM_RR
- wire segments 286 -> 326
Other:
- moved on the sheet: C1, C11, C12, C2, C3, C4, C?, D1, D2, D?, J1, J2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
