File: integrator.sch (KiCad schematic (older format))
At the start: 94 parts, among them J1 SJ-3524-SMT, J2 SJ-3524-SMT, J3 SP-3533-02, J4 SP-3533-02, J5 USB4105-GF-A, J6 Conn_ARM_JTAG_SWD_10, J7 test point, SW1 EVQP40B3M, SW2 EVQP40B3M, SW3 EVQP40B3M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

Commit message: moved logos, misc tweaks
Changed lines of the file:
@@
 Text GLabel 9900 6950 2    50   Input ~ 0
 sw2
-Text GLabel 7250 5050 0    50   Input ~ 0
+Text GLabel 7250 4950 0    50   Input ~ 0
 sw3
 Text GLabel 7250 5450 0    50   Input ~ 0
@@
 Text GLabel 7250 5250 0    50   BiDi ~ 0
 po_swdio
-Text GLabel 7250 4950 0    50   Input ~ 0
+Text GLabel 7250 5050 0    50   Input ~ 0
 po_swo
 Text GLabel 7250 5350 0    50   Input ~ 0

Commit message: resistor tweaks
Parts:
- R15: value 1k -> 1k 5%
- R17: value 100 1% -> 100 1%
- R6: value 4.7k -> 5.1k
Changed lines of the file:
@@
 P 13000 7150
 F 0 "R6" H 13070 7196 50  0000 L CNN
-F 1 "4.7k" H 13070 7105 50  0000 L CNN
+F 1 "5.1k" H 13070 7105 50  0000 L CNN
 F 2 "Resistor_SMD:R_0805_2012Metric" V 12930 7150 50  0001 C CNN
 F 3 "~" H 13000 7150 50  0001 C CNN
@@
 P 7300 3550
 F 0 "R15" V 7093 3550 50  0000 C CNN
-F 1 "1k" V 7184 3550 50  0000 C CNN
+F 1 "1k 5%" V 7184 3550 50  0000 C CNN
 F 2 "Resistor_SMD:R_0805_2012Metric" V 7230 3550 50  0001 C CNN
 F 3 "~" H 7300 3550 50  0001 C CNN
@@
 P 13550 2500
 F 0 "R17" H 13400 2450 50  0000 C CNN
-F 1 "100  1%" H 13400 2550 50  0000 C CNN
+F 1 "100 1%" H 13400 2550 50  0000 C CNN
 F 2 "Resistor_SMD:R_0805_2012Metric" V 13480 2500 50  0001 C CNN
 F 3 "~" H 13550 2500 50  0001 C CNN

Commit message: v9 checkpoint/wip
Parts:
- removed C31: 0.1uf, Capacitor_SMD:C_0805_2012Metric, symbol Device:C_Small
- removed C35: 1uf ceramic, Capacitor_SMD:C_0805_2012Metric, symbol Device:C_Small
- removed U2: MCP1700-2302E/TT, Package_TO_SOT_SMD:SOT-23, symbol Regulator_Linear:MCP1700-2502E_SOT23
- added C?: 0.1uf ceramic, Capacitor_SMD:C_0805_2012Metric, symbol Device:C_Small
- added D?: 200mv drop, Diode_SMD:D_SMB, symbol Device:D_Schottky_Small
- added R?: 100k, Resistor_SMD:R_0805_2012Metric, symbol Device:R
- added R?: 220k, Resistor_SMD:R_0805_2012Metric, symbol Device:R
- added U?: XC6501D331NR-G, SSOT-24_TOR, symbol XC6501D331NR-G:XC6501D331NR-G
Connections:
- net labels added: VAbuf, VUSB
- net labels removed: VAref
- wire segments 433 -> 441
Other:
- note added: "+1.8-3.3V"
- note added: "+2.0-2.5V"
- note added: "+3.3V \nUSB+ REGULATOR"
- note removed: "+2.5V"
- moved on the sheet: C1, C15, C16, C28, C3, C5, D1, D3, J5, J7, JP11, JP6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

Commit message: v9 schematic updates
Parts:
- removed J3, J4: SP-3533-02, SP-3533-02:CUI_SP-3533-02, symbol SP-3533-02:SP-3533-02
- added C35: 0.1uf, Capacitor_SMD:C_0805_2012Metric, symbol Device:C_Small
- added D2: <100mv drop, Diode_SMD:D_SMB, symbol Device:D_Schottky_Small
- LED1, LED2, LED3, LED4: value LS_L29K-G1J2-1-Z -> CSL1901VW1
- gave numbers to parts that had none: 5
Connections:
- net Earth: now also C35.2
- net VRaw: now also D2.1 (K)
- net VReg: no longer J6.1 (VTref)
- net VUSB: now also C35.1
- net pi_swo: now reaches J6.6 (SWO/TDO)
- net pi_swo: now also U5.27 (GPIO16)
- new net: D2.2 (A), J6.1 (VTref)
- no-connect marks 17 -> 15
Other:
- note removed: "3.5mm\nBRIDGE\nCONNECTOR\n(OPTIONAL)"
Changed lines of the file:
@@
 P 14750 800
 F 0 "LED2" H 14950 625 60  0000 C CNN
-F 1 "LS_L29K-G1J2-1-Z" H 14950 500 60  0000 C CNN
+F 1 "CSL1901VW1" H 14950 500 60  0000 C CNN
 F 2 "LED_SMD:LED_0603_1608Metric" H 14950 440 60  0001 C CNN
 F 3 "" H 14750 800 60  0000 C CNN
@@
 P 8650 1100
 F 0 "LED3" H 8850 925 60  0000 C CNN
-F 1 "LS_L29K-G1J2-1-Z" H 8850 800 60  0000 C CNN
+F 1 "CSL1901VW1" H 8850 800 60  0000 C CNN
 F 2 "LED_SMD:LED_0603_1608Metric" H 8850 740 60  0001 C CNN
 F 3 "" H 8650 1100 60  0000 C CNN
@@
 P 8150 8600
 F 0 "LED4" H 8350 8425 60  0000 C CNN
-F 1 "LS_L29K-G1J2-1-Z" H 8350 8300 60  0000 C CNN
+F 1 "CSL1901VW1" H 8350 8300 60  0000 C CNN
 F 2 "LED_SMD:LED_0603_1608Metric" H 8350 8240 60  0001 C CNN
 F 3 "" H 8150 8600 60  0000 C CNN
@@
 	6550 7250 6450 7350
 $Comp
-L SP-3533-02:SP-3533-02 J3
-U 1 1 628172FF
-P 10300 8650
-F 0 "J3" V 9653 8420 50  0000 R CNN
-F 1 "SP-3533-02" V 9562 8420 50  0001 R CNN
-F 2 "SP-3533-02:CUI_SP-3533-02" H 10300 8650 50  0001 L BNN
-F 3 "" H 10300 8650 50  0001 L BNN
-F 4 "Manufacturer Recommendations" H 10300 8650 50  0001 L BNN "STANDARD"
-F 5 "1.01" H 10300 8650 50  0001 L BNN "PARTREV"
-F 6 "5.0mm" H 10300 8650 50  0001 L BNN "MAXIMUM_PACKAGE_HEIGHT"
-F 7 "CUI Devices" H 10300 8650 50  0001 L BNN "MANUFACTURER"
-	1    10300 8650
-	0    -1   -1   0
-$EndComp
-$Comp
 L power:Earth #PWR0126
 U 1 1 62D85090
@@
 P 2400 950
 F 0 "LED1" H 2600 775 60  0000 C CNN
-F 1 "LS_L29K-G1J2-1-Z" H 2600 650 60  0000 C CNN
+F 1 "CSL1901VW1" H 2600 650 60  0000 C CNN
 F 2 "LED_SMD:LED_0603_1608Metric" H 2600 590 60  0001 C CNN
 F 3 "" H 2400 950 60  0000 C CNN
@@
 Wire Wire Line
 	2000 950  1900 1050
-$Comp
-L SP-3533-02:SP-3533-02 J4
-U 1 1 6285D1EA
-P 10900 8650
-F 0 "J4" V 10253 8420 50  0000 R CNN
-F 1 "SP-3533-02" V 10162 8420 50  0000 R CNN
-F 2 "SP-3533-02:CUI_SP-3533-02" H 10900 8650 50  0001 L BNN
-F 3 "" H 10900 8650 50  0001 L BNN
-F 4 "Manufacturer Recommendations" H 10900 8650 50  0001 L BNN "STANDARD"
-F 5 "1.01" H 10900 8650 50  0001 L BNN "PARTREV"
-F 6 "5.0mm" H 10900 8650 50  0001 L BNN "MAXIMUM_PACKAGE_HEIGHT"
-F 7 "CUI Devices" H 10900 8650 50  0001 L BNN "MANUFACTURER"
-	1    10900 8650
-	0    -1   -1   0
-$EndComp
 Wire Wire Line
 	1900 9600 2150 9600
@@
 $EndComp
 Connection ~ 13250 7850
-Wire Wire Line
-	10200 8550 10200 8450
-Wire Wire Line
-	10200 8450 10800 8450
-Wire Wire Line
-	10800 8450 10800 8550
-Wire Wire Line
-	10300 8550 10300 8400
-Wire Wire Line
-	10300 8400 10900 8400
-Wire Wire Line
-	10900 8400 10900 8550
-Wire Wire Line
-	10400 8550 10400 8350
 Wire Wire Line
 	5300 -6550 5900 -6550
@@
 Text GLabel 7300 7150 0    50   Input ~ 0
 pi_swclk
-Text GLabel 7300 7250 0    50   Input ~ 0
+Text GLabel 7300 7250 0    50   BiDi ~ 0
 pi_swdio
 Text GLabel 7300 7350 0    50   Input ~ 0
@@
 Wire Wire Line
 	12850 5100 12900 5100
-Text GLabel 12850 5100 0    50   Output ~ 0
+Text GLabel 12850 5100 0    50   BiDi ~ 0
 pi_swdio
 Text GLabel 12850 5200 0    50   Output ~ 0
@@
 	-1   0    0    1
 $EndComp
-Text GLabel 13400 5800 3    50   Input ~ 0
-VReg
-Wire Wire Line
-	13400 5700 13400 5800
+Text GLabel 12800 5900 0    50   Output ~ 0
+VRaw
 $Comp
 L SJ-3524-SMT:SJ-3524-SMT J1
@@
 Text Notes 900  6600 0    60   ~ 0
 +2.0-5.0V
-Text Notes 11200 8650 0    60   ~ 0
-3.5mm\nBRIDGE\nCONNECTOR\n(OPTIONAL)
 Text Notes 8800 9250 0    60   ~ 0
 CONFIG/RESET \nBUTTON\n(incomplete)
@@
 experimental\nbypass 2
 Wire Wire Line
-	10400 8350 11000 8350
-Wire Wire Line
 	8050 3750 8000 3750
 Wire Wire Line
@@
 	9900 7150 9800 7150
 NoConn ~ 13750 6950
-NoConn ~ 7400 7450
 NoConn ~ 7400 7550
 NoConn ~ 7400 5650
@@
 	12850 5400 12900 5400
 NoConn ~ 12900 4900
-NoConn ~ 12900 5000
 NoConn ~ 13500 4500
 $Comp
@@
 $EndComp
 $Comp
-L power:Earth #PWR0138
-U 1 1 63D1EA01
-P 11000 8100
-F 0 "#PWR0138" H 11000 7850 50  0001 C CNN
-F 1 "Earth" H 11000 7950 50  0001 C CNN
-F 2 "" H 11000 8100 50  0000 C CNN
-F 3 "" H 11000 8100 50  0000 C CNN
-	1    11000 8100
-	-1   0    0    1
-$EndComp
-$Comp
 L power:Earth #PWR0140
 U 1 1 63D5B706
@@
 Wire Wire Line
 	13900 6750 13750 6750
-Wire Wire Line
-	11000 8100 11000 8350
-Connection ~ 11000 8350
-Wire Wire Line
-	11000 8350 11000 8550
 $Comp
 L Device:C_Small C34
@@
 VReg
 $Comp
-L Device:R R?
+L Device:R R21
 U 1 1 63F92044
 P 14750 7000
-F 0 "R?" H 14820 7046 50  0000 L CNN
+F 0 "R21" H 14820 7046 50  0000 L CNN
 F 1 "100k" H 14820 6955 50  0000 L CNN
 F 2 "Resistor_SMD:R_0805_2012Metric" V 14680 7000 50  0001 C CNN
@@
 $EndComp
 $Comp
-L Device:R R?
+L Device:R R22
 U 1 1 63F92C22
 P 14750 7300
-F 0 "R?" H 14820 7346 50  0000 L CNN
+F 0 "R22" H 14820 7346 50  0000 L CNN
 F 1 "220k" H 14820 7255 50  0000 L CNN
 F 2 "Resistor_SMD:R_0805_2012Metric" V 14680 7300 50  0001 C CNN
@@
 Connection ~ 14750 7150
 $Comp
-L power:Earth #PWR?
+L power:Earth #PWR05
 U 1 1 63FE919B
 P 14600 7500
-F 0 "#PWR?" H 14600 7250 50  0001 C CNN
+F 0 "#PWR05" H 14600 7250 50  0001 C CNN
 F 1 "Earth" H 14600 7350 50  0001 C CNN
 F 2 "" H 14600 7500 50  0000 C CNN
@@
 	1500 4150 2950 4150
 $Comp
-L XC6501D331NR-G:XC6501D331NR-G U?
+L XC6501D331NR-G:XC6501D331NR-G U2
 U 1 1 641D5565
 P 2300 8050
-F 0 "U?" H 3100 8437 60  0000 C CNN
+F 0 "U2" H 3100 8437 60  0000 C CNN
 F 1 "XC6501D331NR-G" H 3100 8331 60  0000 C CNN
 F 2 "SSOT-24_TOR" H 3100 8290 60  0001 C CNN
@@
 Connection ~ 2200 8050
 $Comp
-L power:Earth #PWR?
+L power:Earth #PWR04
 U 1 1 64235625
 P 3700 8400
-F 0 "#PWR?" H 3700 8150 50  0001 C CNN
+F 0 "#PWR04" H 3700 8150 50  0001 C CNN
 F 1 "Earth" H 3700 8250 50  0001 C CNN
 F 2 "" H 3700 8400 50  0000 C CNN
@@
 	3650 8250 3600 8250
 $Comp
-L Device:C_Small C?
+L Device:C_Small C31
 U 1 1 64294B85
 P 2300 7850
-F 0 "C?" H 2392 7896 50  0000 L CNN
+F 0 "C31" H 2392 7896 50  0000 L CNN
 F 1 "0.1uf ceramic" H 2392 7805 50  0000 L CNN
 F 2 "Capacitor_SMD:C_0805_2012Metric" H 2300 7850 50  0001 C CNN
@@
 $EndComp
 $Comp
-L power:Earth #PWR?
+L power:Earth #PWR03
 U 1 1 64294B8F
 P 2450 7700
-F 0 "#PWR?" H 2450 7450 50  0001 C CNN
+F 0 "#PWR03" H 2450 7450 50  0001 C CNN
 F 1 "Earth" H 2450 7550 50  0001 C CNN
 F 2 "" H 2450 7700 50  0000 C CNN
@@
 Wire Wire Line
 	10600 5650 10600 6150
-Text GLabel 11400 5300 2    50   Input ~ 0
-VUSB
-Wire Wire Line
-	9800 5750 10550 5750
-Wire Wire Line
-	10550 5750 10550 5400
-Wire Wire Line
-	10550 5400 11050 5400
-Wire Wire Line
-	11050 5400 11050 5300
-Wire Wire Line
-	11050 5300 11400 5300
 Wire Wire Line
 	9800 6250 10600 6250
@@
 VAbuf
 $Comp
-L Device:D_Schottky_Small D?
+L Device:D_Schottky_Small D4
 U 1 1 646D3E37
 P 14150 8350
-F 0 "D?" H 14200 8550 50  0000 R CNN
+F 0 "D4" H 14200 8550 50  0000 R CNN
 F 1 "200mv drop" H 14400 8450 50  0000 R CNN
 F 2 "Diode_SMD:D_SMB" V 14150 8350 50  0001 C CNN
@@
 Wire Wire Line
 	13250 8450 13250 8800
+Wire Wire Line
+	13400 5700 13400 5900
+Wire Wire Line
+	13400 5900 13250 5900
+Wire Wire Line
+	12800 5900 13050 5900
+Wire Wire Line
+	9800 5750 10550 5750
+Wire Wire Line
+	10550 5750 10550 5400
+Wire Wire Line
+	11050 5400 11050 5300
+Wire Wire Line
+	10550 5400 11050 5400
+Wire Wire Line
+	11050 5300 11250 5300
+Text GLabel 11400 5300 2    50   Input ~ 0
+VUSB
+$Comp
+L Device:D_Schottky_Small D2
+U 1 1 648DBA37
+P 13150 5900
+F 0 "D2" H 13200 6100 50  0000 R CNN
+F 1 "<100mv drop" H 13400 6000 50  0000 R CNN
+F 2 "Diode_SMD:D_SMB" V 13150 5900 50  0001 C CNN
+F 3 "https://www.vishay.com/docs/95722/vs-10bq015hm3.pdf" V 13150 5900 50  0001 C CNN
+	1    13150 5900
+	1    0    0    -1
+$EndComp
+$Comp
+L Device:C_Small C35
+U 1 1 6499D85A
+P 11250 5400
+F 0 "C35" H 11342 5446 50  0000 L CNN
+F 1 "0.1uf" H 11342 5355 50  0000 L CNN
+F 2 "Capacitor_SMD:C_0805_2012Metric" H 11250 5400 50  0001 C CNN
+F 3 "~" H 11250 5400 50  0001 C CNN
+	1    11250 5400
+	1    0    0    -1
+$EndComp
+Connection ~ 11250 5300
+Wire Wire Line
+	11250 5300 11400 5300
+Wire Wire Line
+	11250 5500 11250 5750
+Text GLabel 7250 7450 0    50   Output ~ 0
+pi_swo
+Wire Wire Line
+	7250 7450 7400 7450
+Text GLabel 12850 5000 0    50   Output ~ 0
+pi_swo
+Wire Wire Line
+	12850 5000 12900 5000
 $EndSCHEMATC

Commit message: v9 checkpoint 2
Parts:
- D2: footprint Diode_SMD:D_SMB -> Diode_SMD:D_0603_1608Metric
- U2: footprint SSOT-24_TOR -> misc:XC6501D331NR-G
Changed lines of the file:
@@
 U 1 1 641D5565
 P 2300 8050
-F 0 "U2" H 3100 8437 60  0000 C CNN
-F 1 "XC6501D331NR-G" H 3100 8331 60  0000 C CNN
-F 2 "SSOT-24_TOR" H 3100 8290 60  0001 C CNN
+F 0 "U2" H 2950 8437 60  0000 C CNN
+F 1 "XC6501D331NR-G" H 2950 8331 60  0000 C CNN
+F 2 "misc:XC6501D331NR-G" H 3100 8290 60  0001 C CNN
 F 3 "" H 2300 8050 60  0000 C CNN
 	1    2300 8050
@@
 F 0 "D2" H 13200 6100 50  0000 R CNN
 F 1 "<100mv drop" H 13400 6000 50  0000 R CNN
-F 2 "Diode_SMD:D_SMB" V 13150 5900 50  0001 C CNN
+F 2 "Diode_SMD:D_0603_1608Metric" V 13150 5900 50  0001 C CNN
 F 3 "https://www.vishay.com/docs/95722/vs-10bq015hm3.pdf" V 13150 5900 50  0001 C CNN
 	1    13150 5900

Commit message: v9 checkpoint 3
Parts:
- removed C9: 1uf ceramic, Capacitor_SMD:C_0805_2012Metric, symbol Device:C_Small
- Y1: MANUFACTURER (none) -> Abracon; MAXIMUM_PACKAGE_HEIGHT (none) -> 4.2 mm; PARTREV (none) -> 02.16.2021; STANDARD (none) -> Manufacturer Recommendations
Changed lines of the file:
@@
 	-1   0    0    1
 $EndComp
-Connection ~ 13250 7850
 Wire Wire Line
 	5300 -6550 5900 -6550
@@
 	13100 7450 13250 7450
 Connection ~ 13250 7450
-Wire Wire Line
-	13250 7450 13250 7850
 $Comp
 L Device:CP1 C16
@@
 F 2 "Crystal:Crystal_SMD_2520-4Pin_2.5x2.0mm" H 5600 6800 50  0001 C CNN
 F 3 "~" H 5600 6800 50  0001 C CNN
+F 4 "Abracon" H 5600 6800 50  0001 C CNN "MANUFACTURER"
+F 5 "4.2 mm" H 5600 6800 50  0001 C CNN "MAXIMUM_PACKAGE_HEIGHT"
+F 6 "02.16.2021" H 5600 6800 50  0001 C CNN "PARTREV"
+F 7 "Manufacturer Recommendations" H 5600 6800 50  0001 C CNN "STANDARD"
 	1    5600 6800
 	0    1    1    0
@@
 	13750 6650 13950 6600
 Wire Wire Line
-	13250 7450 13900 7450
+	13250 7450 13700 7450
 Wire Wire Line
 	13900 7450 13900 6750
@@
 Text Notes 3650 6200 0    60   ~ 0
 +1.8V
-$Comp
-L Device:C_Small C9
-U 1 1 659664DC
-P 14150 7750
-F 0 "C9" H 14242 7796 50  0000 L CNN
-F 1 "1uf ceramic" H 14242 7705 50  0000 L CNN
-F 2 "Capacitor_SMD:C_0805_2012Metric" H 14150 7750 50  0001 C CNN
-F 3 "~" H 14150 7750 50  0001 C CNN
-	1    14150 7750
-	1    0    0    -1
-$EndComp
-$Comp
-L power:Earth #PWR0142
-U 1 1 659664E2
-P 14300 7500
-F 0 "#PWR0142" H 14300 7250 50  0001 C CNN
-F 1 "Earth" H 14300 7350 50  0001 C CNN
-F 2 "" H 14300 7500 50  0000 C CNN
-F 3 "" H 14300 7500 50  0000 C CNN
-	1    14300 7500
-	0    -1   -1   0
-$EndComp
-Wire Wire Line
-	14150 7650 14150 7550
-Wire Wire Line
-	14150 7550 14300 7500
-Connection ~ 14150 7850
 Wire Wire Line
 	13250 8250 13250 7850
@@
 	0    -1   -1   0
 $EndComp
-Text Label 13250 7700 0    50   ~ 0
+Text Label 13700 7650 0    50   ~ 0
 po_batt
 Wire Wire Line
@@
 	14150 8750 14150 8450
 Wire Wire Line
-	13250 7850 14000 7850
+	13250 7850 13700 7850
 Wire Wire Line
 	13250 8450 13250 8800
@@
 Wire Wire Line
 	12850 5000 12900 5000
+Wire Wire Line
+	13700 7450 13700 7850
+Connection ~ 13700 7450
+Wire Wire Line
+	13700 7450 13900 7450
+Connection ~ 13700 7850
+Wire Wire Line
+	13700 7850 14000 7850
 $EndSCHEMATC

Commit message: possibly finished v9
Parts:
- C15, C16: footprint Capacitor_SMD:CP_Elec_6.3x5.2 -> Capacitor_SMD:CP_Elec_5x4.4
- J5: footprint usb4105:GCT_USB4105-GF-A -> misc:HRO_TYPE-C-31-M-12-Paste-Lugs
- U1: footprint Package_TO_SOT_SMD:SOT-23-6_Handsoldering -> Package_TO_SOT_SMD:SOT-23-6
Connections:
- net pi_txin: now reaches J6.8 (NC/TDI)
- net pi_txin: now also U5.28 (GPIO17)
- no-connect marks 15 -> 13
Changed lines of the file:
@@
 F 0 "C15" V 2002 7150 50  0000 C CNN
 F 1 "100uf" V 1911 7150 50  0000 C CNN
-F 2 "Capacitor_SMD:CP_Elec_6.3x5.2" H 1750 7150 50  0001 C CNN
+F 2 "Capacitor_SMD:CP_Elec_5x4.4" H 1750 7150 50  0001 C CNN
 F 3 "~" H 1750 7150 50  0001 C CNN
 	1    1750 7150
@@
 	9900 7150 9800 7150
 NoConn ~ 13750 6950
-NoConn ~ 7400 7550
 NoConn ~ 7400 5650
 NoConn ~ 9800 6450
@@
 Wire Wire Line
 	12850 5400 12900 5400
-NoConn ~ 12900 4900
 NoConn ~ 13500 4500
 $Comp
@@
 F 0 "C16" V 3202 7150 50  0000 C CNN
 F 1 "100uf" V 3111 7150 50  0000 C CNN
-F 2 "Capacitor_SMD:CP_Elec_6.3x5.2" H 2950 7150 50  0001 C CNN
+F 2 "Capacitor_SMD:CP_Elec_5x4.4" H 2950 7150 50  0001 C CNN
 F 3 "~" H 2950 7150 50  0001 C CNN
 	1    2950 7150
@@
 F 0 "U1" H 2900 6915 50  0000 C CNN
 F 1 "XC6415" H 2900 6824 50  0000 C CNN
-F 2 "Package_TO_SOT_SMD:SOT-23-6_Handsoldering" H 2900 6850 50  0001 C CNN
+F 2 "Package_TO_SOT_SMD:SOT-23-6" H 2900 6850 50  0001 C CNN
 F 3 "https://www.torexsemi.com/file/xc6415/XC6415.pdf" H 2900 6850 50  0001 C CNN
 	1    2900 6450
@@
 F 0 "J5" H 2300 5517 50  0000 C CNN
 F 1 "USB4105-GF-A" H 2300 5426 50  0000 C CNN
-F 2 "usb4105:GCT_USB4105-GF-A" H 2300 4850 50  0001 L BNN
+F 2 "misc:HRO_TYPE-C-31-M-12-Paste-Lugs" H 2300 4850 50  0001 L BNN
 F 3 "" H 2300 4850 50  0001 L BNN
 F 4 "A3" H 2300 4850 50  0001 L BNN "PARTREV"
@@
 Wire Wire Line
 	7250 7450 7400 7450
-Text GLabel 12850 5000 0    50   Output ~ 0
+Text GLabel 12850 5000 0    50   Input ~ 0
 pi_swo
 Wire Wire Line
@@
 Wire Wire Line
 	13700 7850 14000 7850
+Text GLabel 7250 7550 0    50   Input ~ 0
+pi_txin
+Wire Wire Line
+	7400 7550 7250 7550
+Text GLabel 12850 4900 0    50   Output ~ 0
+pi_txin
+Wire Wire Line
+	12900 4900 12850 4900
 $EndSCHEMATC
