File: integrator.kicad_pcb (KiCad board)
At the start: 4 copper layers, 65.5 x 117 mm, 102 parts, among them J1 SJ-3524-SMT, J2 SJ-3524-SMT, J3 SP-3533-02, J4 SP-3533-02, J5 USB4105-GF-A, J6 Conn_ARM_JTAG_SWD_10, J7 test point, SW1 EVQP40B3M, SW2 EVQP40B3M, SW3 EVQP40B3M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

Commit message: test points & tweaks
Parts:
- J7: footprint Connector_PinHeader_2.54mm:PinHeader_2x02_P2.54mm_Vertical -> Connector_PinHeader_2.54mm:PinHeader_1x02_P2.54mm_Vertical
- moved REF** 24.9 mm to (130.2, 107.5)
- moved G*** 18.3 mm to (170.3, 152.6)
- moved REF** 17.9 mm to (177.5, 110.8)
- moved G*** 8.65 mm to (153.3, 118.4)
- moved C35 2.33 mm to (129.8, 128.8)
- moved C9 2.33 mm to (130.6, 121.6)
- moved U2 2.33 mm to (129.8, 125.3)
- turned J7 to 0 degrees
Routing:
- net Earth: track 150.0 -> 161.1 mm, vias 72 -> 83
- net VRaw: track 97.0 -> 86.4 mm
- net /po_batt: track 124.0 -> 130.1 mm, vias 4 -> 11
- net po_play: track 117.4 -> 118.6 mm
Other:
- board text added: "Varef"
- board text added: "Vraw"
- board text added: "Vreg"
- board text added: "po_batt"

Commit message: moved logos, misc tweaks
Parts:
- removed the G*** at (170.3, 152.6)
- removed the G*** at (153.3, 118.4)
- removed the REF** at (130.2, 107.5)
- removed the REF** at (177.5, 110.8)
- added G***: LOGO, misc:UKCA logo 5x5mm, F.Cu at (128.1, 158.0)
- added G***: LOGO, misc:glutenfree 5x5mm, F.Cu at (180.7, 158.0)
- added G***: LOGO, misc:CE logo 7x5mm, F.Cu at (140.1, 158.0)
- added G***: LOGO, misc:FCC logo 5x6mm, F.Cu at (172.6, 158.0)
- moved J7 2.53 mm to (133.6, 124.2), turned to 180 degrees
Connections:
- J7 pad 1: VRaw -> /po_batt
- J7 pad 2: /po_batt -> VRaw
- U5 pad 2: po_swo -> sw3
- U5 pad 3: sw3 -> po_swo
Routing:
- net Earth: track 161.1 -> 162.5 mm
- net sw3: track 121.9 -> 120.8 mm, vias 2 -> 0
- net po_play: track 118.6 -> 119.5 mm
- net po_swdio: track 109.1 -> 110.0 mm
- net po_swclk: track 108.2 -> 109.1 mm
- net po_swo: track 114.2 -> 113.4 mm
Other:
- board text added: "DON’T STOP"
- board text added: "NOT STOPPING"

Commit message: tweaks
Parts:
- J5: footprint usb4105:GCT_USB4105-GF-A -> misc:HRO_TYPE-C-31-M-12-Paste-Lugs

Commit message: v9 checkpoint/wip
Routing:
- net VInt: track 25.7 -> 26.2 mm

Commit message: v9 checkpoint 2
Parts:
- added C31: 0.1uf ceramic, Capacitor_SMD:C_0805_2012Metric, B.Cu at (115.5, 126.2)
- added C35: 0.1uf, Capacitor_SMD:C_0805_2012Metric, B.Cu at (115.5, 123.2)
- added D2: <100mv drop, Diode_SMD:D_0603_1608Metric, B.Cu at (166.6, 150.1)
- added D4: 200mv drop, Diode_SMD:D_SMB, B.Cu at (130.4, 125.4)
- added R21: 100k, Resistor_SMD:R_0805_2012Metric, B.Cu at (175.6, 56.9)
- added R22: 220k, Resistor_SMD:R_0805_2012Metric, B.Cu at (179.8, 56.9)
- LED1, LED2, LED3, LED4: value LS_L29K-G1J2-1-Z -> CSL1901VW1
- R15: value 1k -> 1k 5%
- R17: value 100 1% -> 100 1%
- R6: value 4.7k -> 5.1k
- U2: value MCP1700-2302E/TT -> XC6501D331NR-G; footprint Package_TO_SOT_SMD:SOT-23 -> misc:XC6501D331NR-G
- moved U2 30.7 mm to (109.8, 148.6), turned to 0 degrees
- moved C35 22.0 mm to (108.9, 135.7)
- moved C9 5.49 mm to (126.5, 118.0)
- moved J7 2.60 mm to (133.4, 126.8), turned to 0 degrees
- moved C22 0.83 mm to (158.1, 126.9)
- moved C21 0.81 mm to (158.1, 124.9)
Connections:
- C3 pad 1: VAref -> VAbuf
- C31 pad 1: VAref -> VAbuf
- J6 pad 1: VReg -> Net-(D2-Pad2)
- J6 pad 6: Net-(J6-Pad6) -> pi_swo
- J7 pad 1: /po_batt -> VAbuf
- J7 pad 2: VRaw -> /po_batt
- JP7 pad 2: VAref -> VAbuf
- JP8 pad 1: VAref -> VAbuf
- POGO1 pad 6: po_wake -> Net-(POGO1-Pad6)
- U1 pad 4: VAref -> VAbuf
- U2 pad 1: Earth -> VRaw
- U2 pad 2: /po_batt -> Earth
- U2 pad 3: VRaw -> VUSB
- U5 pad 27: Net-(U5-Pad27) -> pi_swo
- U5 pad 43: VAref -> VReg
- U5 pad 48: VReg -> VUSB
- Y1 pad 2: Earth -> Net-(C11-Pad1)
- Y1 pad 3: Net-(C11-Pad1) -> (no net)
- Y1 pad 4: Earth -> (no net)
Routing:
- net VAref: track 97.7 -> 0.00 mm, vias 18 -> 0
- net VAbuf: track 0.00 -> 97.7 mm, vias 0 -> 18
- net pi_swo: track 0.00 -> 30.7 mm, vias 0 -> 2
- net Net-(D2-Pad2): track 0.00 -> 30.3 mm, vias 0 -> 4
- net Net-(POGO1-Pad6): track 0.00 -> 29.3 mm
- net VReg: track 204.0 -> 184.0 mm
- net po_wake: track 120.5 -> 104.0 mm
- net VRaw: track 86.4 -> 99.4 mm, vias 0 -> 8
- net /po_batt: track 130.1 -> 121.0 mm
- net Earth: track 162.5 -> 155.3 mm, vias 83 -> 76
- net VInt: track 26.2 -> 27.2 mm
- net ring1: track 24.4 -> 24.9 mm
- net pi_swdio: track 26.1 -> 26.7 mm
Other:
- board text added: "VAbuf"
- board text removed: "Varef"

Commit message: v9 checkpoint 3
Parts:
- removed the C35 at (108.9, 135.7)
- removed C9: 1uf ceramic, Capacitor_SMD:C_0805_2012Metric
- removed J3, J4: SP-3533-02, SP-3533-02:CUI_SP-3533-02
- removed REF** (x4): mousebites_sparkfun, misc:mousebites_sparkfun
- U2: value XC6501D331NR-G -> SSOT-24_TOR
- moved C35 47.6 mm to (158.3, 144.0)
- moved U2 24.5 mm to (133.7, 143.4)
- moved C31 23.3 mm to (131.2, 143.4), turned to 90 degrees
- moved D4 1.00 mm to (129.4, 125.4)
- moved C26 0.48 mm to (153.9, 142.7)
- moved C27 0.48 mm to (151.8, 142.7)
- moved C29 0.48 mm to (149.8, 142.7)
- moved J7 0.18 mm to (133.6, 126.8)
- turned JP11 to 0 degrees
Connections:
- Y1 pad 2: Net-(C11-Pad1) -> (no net)
- Y1 pad 3: (no net) -> Net-(C11-Pad1)
Routing:
- net VAbuf: track 97.7 -> 139.8 mm, vias 18 -> 22
- net VUSB: track 0.00 -> 39.3 mm, vias 0 -> 7
- net VRaw: track 99.4 -> 113.4 mm
- net Net-(J3-Pad2): track 11.1 -> 0.00 mm
- net Net-(J3-Pad1): track 11.1 -> 0.00 mm
- net VReg: track 184.0 -> 180.2 mm
- net Earth: track 155.3 -> 153.5 mm, vias 76 -> 84
- net VInt: track 27.2 -> 27.9 mm
Other:
- outline, holes or cut-outs redrawn
- board text removed: "JLCJLCJLCJLC"
- board text removed: "Vraw"

Commit message: possibly finished v9
Parts:
- removed the C31 at (161.0, 140.3)
- C15, C16: footprint Capacitor_SMD:CP_Elec_6.3x5.2 -> Capacitor_SMD:CP_Elec_5x4.4
- U1: footprint Package_TO_SOT_SMD:SOT-23-6_Handsoldering -> Package_TO_SOT_SMD:SOT-23-6
- U2: value SSOT-24_TOR -> XC6501D331NR-G
- moved R21 10.9 mm to (178.6, 67.3), turned to 90 degrees
- moved R22 10.5 mm to (180.6, 67.3), turned to 270 degrees
- moved R1 0.25 mm to (157.5, 149.5)
- moved R2 0.25 mm to (150.6, 149.5)
- moved R3 0.25 mm to (155.0, 149.5)
- moved R7 0.25 mm to (153.0, 149.5)
Connections:
- J6 pad 8: Net-(J6-Pad8) -> pi_txin
- U5 pad 28: Net-(U5-Pad28) -> pi_txin
Routing:
- net pi_txin: track 0.00 -> 35.8 mm, vias 0 -> 1
- net po_wake: track 104.0 -> 92.2 mm
- net VAbuf: track 139.8 -> 128.7 mm
- net AGnd: track 37.1 -> 32.9 mm, vias 7 -> 10
- net Earth: track 153.5 -> 156.7 mm, vias 84 -> 87
- net Net-(POGO1-Pad6): track 29.3 -> 31.8 mm
- net Net-(JP10-Pad2): track 76.6 -> 78.7 mm
- net /po_batt: track 121.3 -> 123.1 mm, vias 11 -> 12
- net Net-(D3-Pad2): track 27.5 -> 29.1 mm
Other:
- board text added: "L"
- board text added: "M"
- board text added: "NOT STOPPING!"
- board text added: "Pocket Integrator"
- board text added: "S"
- board text added: "VUSB"
- board text added: "Version 9 Release Candidate Feb 2023"
- board text added: "bit.ly/pocketintegrator"
- board text removed: "MSL"
- board text removed: "NOT STOPPING"
- board text removed: "Pocket Integrator bit.ly/pocketintegrator"

Commit message: sysclk testpad, jmpr cleanup
Parts:
- hr enable: renamed from JP10
- moved JP7 0.50 mm to (160.7, 117.3)
- moved JP8 0.50 mm to (172.2, 117.3)
- moved C25 0.45 mm to (161.4, 136.6)
- moved C24 0.36 mm to (161.5, 132.3)
- renumbered JP6 to GND, JP1 to bootsel
Routing:
- net Net-(U5-Pad37): track 0.00 -> 10.1 mm
- net Net-(C32-Pad1): track 14.1 -> 16.6 mm
- net Aref_enable: track 36.1 -> 34.3 mm
- net po_wake: track 92.2 -> 93.6 mm
- net VUSB: track 39.3 -> 37.9 mm
- net tip1: track 28.2 -> 27.4 mm
- net VAbuf: track 128.7 -> 129.5 mm
- added copper zone on B.Cu, net Net-(U5-Pad37)
Other:
- board text added: "clk_sys gpio25"
